File: Shunt Resistor Array.kicad_sch (KiCad schematic)
At the start: 10 parts

Commit message: Most work done
Parts:
- renumbered R9 to R10, R10 to R11, R11 to R12, R12 to R13, R13 to R14, R14 to R15, R15 to R16, R16 to R17, R7 to R8, R8 to R9
