File: [EXOTIC] AVR Kit.kicad_sch (KiCad schematic)
At the start: 18 parts, among them J2 AVR-ISP-10, J3 USB_B, J4 Conn_01x08_Socket, J5 Conn_01x08_Socket, J6 Conn_01x09_Socket, J7 Conn_01x07_Socket, SW1 SW_Push, U1 ATmega32A-P, U6 CH340C, Y1 16 MHz

Commit message: Delete ibom.html
Parts:
- J3: Local Seller https://makerselectronics.com/product/chip-resistor-smd-330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 -> https://makerselectronics.com/product/usb-connector-on-pcb-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
Changed lines of the file:
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@@
       (effects (font (size 1.27 1.27)) hide)
     )
-    (property "Local Seller" "https://makerselectronics.com/product/chip-resistor-smd-330k%cf%89-%c2%b11-250mw-1206" (at 199.39 102.87 0)
+    (property "Local Seller" "https://makerselectronics.com/product/usb-connector-on-pcb-b-type-female" (at 199.39 102.87 0)
       (effects (font (size 1.27 1.27)) hide)
     )

Commit message: Schematic Revision C2
Parts:
- J4, J5, J6, J7: Local Seller (none) -> https://makerselectronics.com/product/pin-headers-female-2-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
Changed lines of the file:
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@@
+      (effects (font (size 1.27 1.27)) hide)
+    )
+    (property "Local Seller" "https://makerselectronics.com/product/pin-headers-female-2-54mm-40-pin-straight-black-11mm" (at 110.49 83.82 0)
       (effects (font (size 1.27 1.27)) hide)
     )
@@
     )
     (property "Datasheet" "~" (at 110.49 106.68 0)
+      (effects (font (size 1.27 1.27)) hide)
+    )
+    (property "Local Seller" "https://makerselectronics.com/product/pin-headers-female-2-54mm-40-pin-straight-black-11mm" (at 110.49 106.68 0)
       (effects (font (size 1.27 1.27)) hide)
     )
@@
       (effects (font (size 1.27 1.27)) hide)
     )
+    (property "Local Seller" "https://makerselectronics.com/product/pin-headers-female-2-54mm-40-pin-straight-black-11mm" (at 110.49 60.96 0)
+      (effects (font (size 1.27 1.27)) hide)
+    )
     (pin "1")
     (pin "2")
@@
       (effects (font (size 1.27 1.27)) hide)
     )
+    (property "Local Seller" "https://makerselectronics.com/product/pin-headers-female-2-54mm-40-pin-straight-black-11mm" (at 110.49 129.54 0)
+      (effects (font (size 1.27 1.27)) hide)
+    )

Commit message: WIP2
Parts:
- added C11: 10 µF, Capacitor_SMD:C_1206_3216Metric_Pad1.33x1.80mm_HandSolder, symbol Device:C_Polarized
- added C12: 100 nF, Capacitor_SMD:C_1206_3216Metric_Pad1.33x1.80mm_HandSolder, symbol Device:C
- Y1: footprint Crystal:Crystal_HC49-4H_Vertical -> M's Library:Crystal_HC49-4H_Vertical_Centered
Connections:
- net GND: now also C11.2, C12.1
- net VBUS: now also C11.1, C12.2
- net at C2.1, U1.12 (XTAL2): now also Y1.2; no longer Y1.1
- net at C1.2, U1.13 (XTAL1): now also Y1.1; no longer Y1.2
Other:
- moved on the sheet: Y1

Commit message: Most work done
Parts:
- U1: footprint M's Library:ZIF Socket 40 Circular Pads -> M's Library:ZIF_Socket_40_Circular_Pads
Connections:
- net GND: now also SW1.2; no longer SW1.1
- net ~{RESET}: now also SW1.1; no longer SW1.2
Changed lines of the file:
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@@
     )
   )
-  (symbol (lib_id "Switch:SW_Push") (at 53.34 44.45 0) (unit 1)
-    (in_bom yes) (on_board yes) (dnp no) (fields_autoplaced)
+  (symbol (lib_id "Switch:SW_Push") (at 53.34 44.45 0) (mirror y) (unit 1)
+    (in_bom yes) (on_board yes) (dnp no)
     (property "Reference" "SW1" (at 53.34 38.1 0)
       (effects (font (size 1.27 1.27)))
@@
       (effects (font (size 1.27 1.27)) (justify left))
     )
-    (property "Footprint" "M's Library:ZIF Socket 40 Circular Pads" (at 76.2 96.52 0)
+    (property "Footprint" "M's Library:ZIF_Socket_40_Circular_Pads" (at 76.2 96.52 0)
       (effects (font (size 1.27 1.27) italic) hide)
     )

Commit message: done something
Parts:
- J3: footprint Connector_USB:USB_B_OST_USB-B1HSxx_Horizontal -> M's Library:USB_B_Connector_Horizontal
Changed lines of the file:
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@@
       (effects (font (size 1.27 1.27)))
     )
-    (property "Footprint" "Connector_USB:USB_B_OST_USB-B1HSxx_Horizontal" (at 195.58 104.14 0)
+    (property "Footprint" "M's Library:USB_B_Connector_Horizontal" (at 195.58 104.14 0)
       (effects (font (size 1.27 1.27)) hide)
     )
