File: Power Management Circuitry.kicad_sch (KiCad schematic)
At the start: 23 parts, among them J1 Barrel_Jack_Switch, Q1 AO3401A, Q2 SI2302, SW2 SW_DPDT_x2, U2 AMS1117-3.3, U3 AMS1117-5.0, U4 LM324, U5 LM339

Commit message: WIP
Parts:
- added R8, R9: 1 Ω, Resistor_THT:R_Axial_DIN0614_L14.3mm_D5.7mm_P7.62mm_Vertical, symbol Device:R
Connections:
- net +5V: now also R8.2, R9.1
- net +5V_{OCP}: now also R8.1, R9.2
Other:
- removed sheet Shunt Resistor Array
Changed lines of the file:
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@@
   (junction (at 66.04 40.64) (diameter 0) (color 0 0 0 0)
   )
+  (junction (at 124.46 55.88) (diameter 0) (color 0 0 0 0)
+  )
   (junction (at 52.07 78.74) (diameter 0) (color 0 0 0 0)
   )
@@
   )
   (junction (at 138.43 43.18) (diameter 0) (color 0 0 0 0)
+  )
+  (junction (at 124.46 43.18) (diameter 0) (color 0 0 0 0)
   )
   (junction (at 66.04 71.12) (diameter 0) (color 0 0 0 0)
@@
     (stroke (width 0) (type default))
   )
-  (wire (pts (xy 111.76 55.88) (xy 138.43 55.88))
-    (stroke (width 0) (type default))
-  )
   (wire (pts (xy 157.48 93.98) (xy 160.02 93.98))
     (stroke (width 0) (type default))
@@
     (stroke (width 0) (type default))
   )
+  (wire (pts (xy 111.76 53.34) (xy 111.76 55.88))
+    (stroke (width 0) (type default))
+  )
   (wire (pts (xy 135.89 78.74) (xy 138.43 78.74))
     (stroke (width 0) (type default))
   )
+  (wire (pts (xy 124.46 43.18) (xy 124.46 45.72))
+    (stroke (width 0) (type default))
+  )
   (wire (pts (xy 254 144.78) (xy 254 147.32))
     (stroke (width 0) (type default))
@@
     (stroke (width 0) (type default))
   )
+  (wire (pts (xy 111.76 55.88) (xy 124.46 55.88))
+    (stroke (width 0) (type default))
+  )
   (wire (pts (xy 215.9 46.99) (xy 222.25 46.99))
     (stroke (width 0) (type default))
@@
     (stroke (width 0) (type default))
   )
+  (wire (pts (xy 124.46 55.88) (xy 138.43 55.88))
+    (stroke (width 0) (type default))
+  )
   (wire (pts (xy 219.71 29.21) (xy 222.25 29.21))
     (stroke (width 0) (type default))
@@
     (stroke (width 0) (type default))
   )
+  (wire (pts (xy 111.76 43.18) (xy 124.46 43.18))
+    (stroke (width 0) (type default))
+  )
   (wire (pts (xy 213.36 52.07) (xy 215.9 52.07))
     (stroke (width 0) (type default))
@@
     (stroke (width 0) (type default))
   )
-  (wire (pts (xy 111.76 43.18) (xy 138.43 43.18))
-    (stroke (width 0) (type default))
-  )
   (wire (pts (xy 138.43 78.74) (xy 138.43 80.01))
     (stroke (width 0) (type default))
@@
     (stroke (width 0) (type default))
   )
+  (wire (pts (xy 124.46 53.34) (xy 124.46 55.88))
+    (stroke (width 0) (type default))
+  )
+  (wire (pts (xy 124.46 43.18) (xy 138.43 43.18))
+    (stroke (width 0) (type default))
+  )
   (wire (pts (xy 236.22 57.15) (xy 238.76 57.15))
     (stroke (width 0) (type default))
@@
   )
   (wire (pts (xy 172.72 151.13) (xy 175.26 151.13))
+    (stroke (width 0) (type default))
+  )
+  (wire (pts (xy 111.76 45.72) (xy 111.76 43.18))
     (stroke (width 0) (type default))
   )
@@
     )
   )
+  (symbol (lib_id "Device:R") (at 124.46 49.53 180) (unit 1)
+    (in_bom yes) (on_board yes) (dnp no) (fields_autoplaced)
+    (property "Reference" "R9" (at 127 48.26 0)
+      (effects (font (size 1.27 1.27)) (justify right))
+    )
+    (property "Value" "1 Ω" (at 127 50.8 0)
+      (effects (font (size 1.27 1.27)) (justify right))
+    )
+    (property "Footprint" "Resistor_THT:R_Axial_DIN0614_L14.3mm_D5.7mm_P7.62mm_Vertical" (at 126.238 49.53 90)
+      (effects (font (size 1.27 1.27)) hide)
+    )
+    (property "Datasheet" "~" (at 124.46 49.53 0)
+      (effects (font (size 1.27 1.27)) hide)
+    )
+    (pin "1")
+    (pin "2")
+    (instances
+      (project "[EXOTIC] AVR Kit"
+        (path "/bd689b4b-40d7-46ba-91b6-965ce30f8212/9da448d2-dd3c-46c7-b716-b331cd5a4621"
+          (reference "R9") (unit 1)
+        )
+      )
+    )
+  )
   (symbol (lib_id "power:+3V3") (at 66.04 68.58 0) (unit 1)
     (in_bom yes) (on_board yes) (dnp no) (fields_autoplaced)
@@
     )
   )
+  (symbol (lib_id "Device:R") (at 111.76 49.53 0) (unit 1)
+    (in_bom yes) (on_board yes) (dnp no) (fields_autoplaced)
+    (property "Reference" "R8" (at 114.3 48.26 0)
+      (effects (font (size 1.27 1.27)) (justify left))
+    )
+    (property "Value" "1 Ω" (at 114.3 50.8 0)
+      (effects (font (size 1.27 1.27)) (justify left))
+    )
+    (property "Footprint" "Resistor_THT:R_Axial_DIN0614_L14.3mm_D5.7mm_P7.62mm_Vertical" (at 109.982 49.53 90)
+      (effects (font (size 1.27 1.27)) hide)
+    )
+    (property "Datasheet" "~" (at 111.76 49.53 0)
+      (effects (font (size 1.27 1.27)) hide)
+    )
+    (pin "1")
+    (pin "2")
+    (instances
+      (project "[EXOTIC] AVR Kit"
+        (path "/bd689b4b-40d7-46ba-91b6-965ce30f8212/9da448d2-dd3c-46c7-b716-b331cd5a4621"
+          (reference "R8") (unit 1)
+        )
+      )
+    )
+  )
   (symbol (lib_id "power:PWR_FLAG") (at 241.3 147.32 180) (unit 1)
     (in_bom yes) (on_board yes) (dnp no) (fields_autoplaced)
@@
       )
     )
-  )
-  (sheet (at 99.06 39.37) (size 12.7 20.32) (fields_autoplaced)
-    (stroke (width 0.1524) (type solid))
-    (fill (color 0 0 0 0.0000))
-    (property "Sheetname" "Shunt Resistor Array" (at 99.06 38.6584 0)
-      (effects (font (size 1.27 1.27)) (justify left bottom))
-    )
-    (property "Sheetfile" "Shunt Resistor Array.kicad_sch" (at 99.06 60.2746 0)
-      (effects (font (size 1.27 1.27)) (justify left top))
-    )
-    (pin "R_Shunt_1" input (at 111.76 43.18 0)
-      (effects (font (size 1.27 1.27)) (justify right))
-    )
-    (pin "R_Shunt_2" input (at 111.76 55.88 0)
-      (effects (font (size 1.27 1.27)) (justify right))
-    )
-    (instances
-      (project "[EXOTIC] AVR Kit"
-        (path "/bd689b4b-40d7-46ba-91b6-965ce30f8212/9da448d2-dd3c-46c7-b716-b331cd5a4621" (page "4"))
-      )
-    )

Commit message: Rev 3.1
Parts:
- removed R4: 6.8 kΩ, Resistor_SMD:R_1206_3216Metric_Pad1.30x1.75mm_HandSolder, symbol Device:R
- added R10 (x2): 0 Ω, Resistor_SMD:R_1206_3216Metric_Pad1.30x1.75mm_HandSolder, symbol Device:R
- D1: footprint LED_THT:LED_D5.0mm_Clear -> LED_SMD:LED_1206_3216Metric_Pad1.42x1.75mm_HandSolder
- renumbered R7 to R6, R8 to R7, R9 to R8
Connections:
- net +3V3: now also R10.1; no longer U5.8 (-)
- net +V_{In}: no longer R4.2
- net GND: now also R4.1
- net at U5.9 (+): now also J1.1, R4.2, SW2.6 (C); no longer R4.1
- net at F1.1: now also SW2.5 (B); no longer SW2.6 (C)
- new net: R10.2, R10.2
- new net: R10.1, U5.8 (-)
Other:
- moved on the sheet: R4, SW2B
