File: Power Management Circuitry.kicad_sch (KiCad schematic)
At the start: 19 parts, among them J1 Barrel_Jack_Switch, J8 5V Headers, J9 3.3 V Headers, Q1 AO3401A, SW2 SW_DPDT_x2, U2 AMS1117-3.3, U3 AMS1117-5.0, U4 LM324

Commit message: Rev 3.99
Parts:
- removed U4: LM324, Package_SO:SO-14_3.9x8.65mm_P1.27mm, symbol Amplifier_Operational:LM324
- added D2: LED, LED_SMD:LED_1206_3216Metric_Pad1.42x1.75mm_HandSolder, symbol Device:LED
- added F2: Polyfuse_Small, Capacitor_THT:C_Disc_D10.5mm_W5.0mm_P5.00mm, symbol Device:Polyfuse_Small
- added JP1: PPTC Bypass, Jumper:SolderJumper-2_P1.3mm_Open_RoundedPad1.0x1.5mm, symbol Jumper:SolderJumper_2_Open
- added R4, R8: 1 kΩ, Resistor_SMD:R_1206_3216Metric_Pad1.30x1.75mm_HandSolder, symbol Device:R
- added U4: LM339, Package_SO:SOIC-14_3.9x8.7mm_P1.27mm, symbol Comparator:LM339
- J8, J9: Local Seller (none) -> https://makerselectronics.com/product/pin-headers-female-2-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
Connections:
- net -V_{In} is gone; now on net GND: C5.2, C6.2, C7.2, C8.2, J1.2, U2.1 (GND), U3.1 (GND)
- net +5V: now also F2.1, JP1.2 (B), R4.2, U4.3 (V+)
- net +5V_{PPTC}: now also F2.2, JP1.1 (A)
- net +V_{In}: now also D2.2 (A), U4.5 (+)
- net GND: now also R8.2, U4.12 (V-)
- net at Q1.1 (G): now also R4.1, U4.2
- net at R11.2: now also U4.4 (-)
- new net: D2.1 (K), R8.1
Other:
- note removed: "Over Current Protection"

Commit message: Rev. L4.2
Parts:
- removed J8: 5V Headers, Connector_PinSocket_2.54mm:PinSocket_1x04_P2.54mm_Vertical, symbol Connector:Conn_01x04_Socket
- added J11: 5 V Headers, Connector_PinSocket_2.54mm:PinSocket_2x04_P2.54mm_Vertical, symbol Connector_Generic:Conn_02x04_Odd_Even
- renumbered C7 to C6, C6 to C7, R4 to R2, R11 to R3, R11 to R4, R11 to R6, R4 to R7, U3 to U2, U2 to U3
Connections:
- net +5V: now also JP1.1 (A), J11.1 (Pin_1), J11.2 (Pin_2), J11.3 (Pin_3), J11.4 (Pin_4); no longer JP1.2 (B)
- net +5V_{PPTC}: now also JP1.2 (B); no longer JP1.1 (A)
- net +V_{In}: now also F1.1; no longer F1.2
- net GND: now also J11.5 (Pin_5), J11.6 (Pin_6), J11.7 (Pin_7), J11.8 (Pin_8)
- net at SW2.2 (B): now also F1.2; no longer F1.1
Other:
- note added: "DC-In Power LED Indicator"
- note added: "Net Tie"
- note removed: "To Do: ~Priority Switch to select which 5V source is the dominant~ DONE"
- note removed: "http://store.logicneed.com/product/20510"
- note removed: "~Two Seperate Op-Amps needed due to difference in power source requirements (Rail selector won't work if the op amp is powered from the +12V)~ DONE"
- moved on the sheet: D2, F1, F2, J9, JP1, Q1, R2, R3, R4, R6, R7, R8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

Commit message: Add files via upload
Parts:
- added H1, H2, H3, H4: MountingHole, MountingHole:MountingHole_2.2mm_M2_Pad, symbol Mechanical:MountingHole
- renumbered J11 to J10
Other:
- note added: "Mounting Holes"
- moved on the sheet: R6
