File: [EXOTIC] AVR Kit.kicad_pcb (KiCad board)
At the start: 2 copper layers, 104.1 x 80 mm, 48 parts, among them J1 Barrel_Jack_Switch, J2 AVR-ISP-10, J3 USB_B, J4 Conn_01x08_Socket, J5 Conn_01x08_Socket, J6 Conn_01x09_Socket, J7 Conn_01x07_Socket, Q1 AO3401A, Q2 SI2302, SW1 SW_Push, SW2 SW_DPDT_x2, U1 ATmega32A-P, U2 AMS1117-5.0, U3 AMS1117-3.3, U4 LM324, U5 LM339, U6 CH340C, Y1 16 MHz

Commit message: Update
Routing:
- net +5V: track 284.1 -> 286.2 mm
- net /MOSI: track 75.0 -> 75.7 mm
- net GND: vias 4 -> 12
Changed lines of the file:
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@@
     (effects (font (size 1 1) (thickness 0.15)))
   )
+  (via (at 151.13 143.51) (size 1.2) (drill 0.6) (layers "F.Cu" "B.Cu") (free) (net 1))
   (via (at 170.18 106.68) (size 1.2) (drill 0.6) (layers "F.Cu" "B.Cu") (free) (net 1))
   (via (at 133.985 102.87) (size 1.2) (drill 0.6) (layers "F.Cu" "B.Cu") (free) (net 1))
-  (via (at 196.85 111.125) (size 1.2) (drill 0.6) (layers "F.Cu" "B.Cu") (free) (net 1))
-  (via (at 198.755 106.045) (size 1.2) (drill 0.6) (layers "F.Cu" "B.Cu") (free) (net 1))
+  (via (at 210.82 111.76) (size 1.2) (drill 0.6) (layers "F.Cu" "B.Cu") (free) (net 1))
+  (via (at 156.21 135.89) (size 1.2) (drill 0.6) (layers "F.Cu" "B.Cu") (free) (net 1))
+  (via (at 199.39 109.22) (size 1.2) (drill 0.6) (layers "F.Cu" "B.Cu") (free) (net 1))
+  (via (at 201.93 135.89) (size 1.2) (drill 0.6) (layers "F.Cu" "B.Cu") (free) (net 1))
+  (via (at 198.755 101.6) (size 1.2) (drill 0.6) (layers "F.Cu" "B.Cu") (free) (net 1))
+  (via (at 176.53 135.89) (size 1.2) (drill 0.6) (layers "F.Cu" "B.Cu") (free) (net 1))
+  (via (at 209.55 119.38) (size 1.2) (drill 0.6) (layers "F.Cu" "B.Cu") (free) (net 1))
+  (via (at 135.89 133.35) (size 1.2) (drill 0.6) (layers "F.Cu" "B.Cu") (free) (net 1))
+  (via (at 176.53 97.79) (size 1.2) (drill 0.6) (layers "F.Cu" "B.Cu") (free) (net 1))
   (segment (start 173.99 121.82) (end 173.99 128.27) (width 0.4) (layer "F.Cu") (net 2))
   (segment (start 172.82 120.65) (end 173.99 121.82) (width 0.4) (layer "F.Cu") (net 2))
@@
   (segment (start 152.4 91.44) (end 149.86 88.9) (width 0.4) (layer "F.Cu") (net 15))
   (segment (start 134.62 88.9) (end 129.54 93.98) (width 0.4) (layer "F.Cu") (net 15))
-  (segment (start 156.21 132.08) (end 190.5 132.08) (width 0.4) (layer "F.Cu") (net 17))
+  (segment (start 148.59 121.92) (end 151.13 124.46) (width 0.4) (layer "F.Cu") (net 17))
+  (segment (start 191.77 130.81) (end 191.77 128.27) (width 0.4) (layer "F.Cu") (net 17))
   (segment (start 191.77 119.38) (end 191.77 128.27) (width 0.4) (layer "F.Cu") (net 17))
-  (segment (start 148.59 121.92) (end 152.4 125.73) (width 0.4) (layer "F.Cu") (net 17))
-  (segment (start 191.77 130.81) (end 191.77 128.27) (width 0.4) (layer "F.Cu") (net 17))
   (segment (start 142.24 123.825) (end 144.145 121.92) (width 0.4) (layer "F.Cu") (net 17))
+  (segment (start 151.13 128.27) (end 154.94 132.08) (width 0.4) (layer "F.Cu") (net 17))
+  (segment (start 151.13 124.46) (end 151.13 128.27) (width 0.4) (layer "F.Cu") (net 17))
   (segment (start 190.5 132.08) (end 191.77 130.81) (width 0.4) (layer "F.Cu") (net 17))
-  (segment (start 152.4 125.73) (end 152.4 128.27) (width 0.4) (layer "F.Cu") (net 17))
+  (segment (start 144.145 121.92) (end 148.59 121.92) (width 0.4) (layer "F.Cu") (net 17))
   (segment (start 142.24 130.81) (end 142.24 123.825) (width 0.4) (layer "F.Cu") (net 17))
-  (segment (start 152.4 128.27) (end 156.21 132.08) (width 0.4) (layer "F.Cu") (net 17))
-  (segment (start 144.145 121.92) (end 148.59 121.92) (width 0.4) (layer "F.Cu") (net 17))
+  (segment (start 154.94 132.08) (end 190.5 132.08) (width 0.4) (layer "F.Cu") (net 17))
   (segment (start 181.61 119.38) (end 181.61 128.27) (width 0.4) (layer "F.Cu") (net 18))
   (segment (start 189.23 111.76) (end 181.61 119.38) (width 0.4) (layer "F.Cu") (net 18))
@@
   (via (at 196.85 109.22) (size 1.2) (drill 0.6) (layers "F.Cu" "B.Cu") (net 18))
   (via (at 132.08 102.87) (size 1.2) (drill 0.6) (layers "F.Cu" "B.Cu") (net 18))
-  (segment (start 147.32 130.81) (end 153.67 137.16) (width 0.4) (layer "B.Cu") (net 18))
-  (segment (start 181.61 134.62) (end 181.61 128.27) (width 0.4) (layer "B.Cu") (net 18))
   (segment (start 184.15 88.9) (end 190.5 95.25) (width 0.4) (layer "B.Cu") (net 18))
-  (segment (start 153.67 137.16) (end 179.07 137.16) (width 0.4) (layer "B.Cu") (net 18))
   (segment (start 144.78 130.81) (end 147.32 130.81) (width 0.4) (layer "B.Cu") (net 18))
+  (segment (start 147.32 130.81) (end 156.21 139.7) (width 0.4) (layer "B.Cu") (net 18))
   (segment (start 165.1 88.9) (end 184.15 88.9) (width 0.4) (layer "B.Cu") (net 18))
   (segment (start 132.08 93.98) (end 135.89 90.17) (width 0.4) (layer "B.Cu") (net 18))
+  (segment (start 181.61 134.62) (end 181.61 128.27) (width 0.4) (layer "B.Cu") (net 18))
   (segment (start 151.13 91.44) (end 162.56 91.44) (width 0.4) (layer "B.Cu") (net 18))
+  (segment (start 176.53 139.7) (end 181.61 134.62) (width 0.4) (layer "B.Cu") (net 18))
   (segment (start 132.08 102.87) (end 132.08 93.98) (width 0.4) (layer "B.Cu") (net 18))
   (segment (start 162.56 91.44) (end 165.1 88.9) (width 0.4) (layer "B.Cu") (net 18))
   (segment (start 196.85 109.22) (end 196.85 96.52) (width 0.4) (layer "B.Cu") (net 18))
-  (segment (start 179.07 137.16) (end 181.61 134.62) (width 0.4) (layer "B.Cu") (net 18))
   (segment (start 149.86 90.17) (end 151.13 91.44) (width 0.4) (layer "B.Cu") (net 18))
+  (segment (start 156.21 139.7) (end 176.53 139.7) (width 0.4) (layer "B.Cu") (net 18))
   (segment (start 135.89 90.17) (end 149.86 90.17) (width 0.4) (layer "B.Cu") (net 18))
   (segment (start 144.78 147.32) (end 148.59 147.32) (width 0.4) (layer "F.Cu") (net 20))
@@
       )
     )
+  )
+  (zone (net 0) (net_name "") (layers "F&B.Cu") (name "Logo") (hatch edge 0.5)
+    (connect_pads (clearance 0))
+    (min_thickness 0.25) (filled_areas_thickness no)
+    (keepout (tracks allowed) (vias not_allowed) (pads allowed) (copperpour allowed) (footprints not_allowed))
+    (fill (thermal_gap 0.5) (thermal_bridge_width 0.5))
+    (polygon
+      (pts
+        (xy 229.87 163.83)
+        (xy 229.87 148.59)
+        (xy 210.82 148.59)
+        (xy 210.82 156.21)
+        (xy 179.07 156.21)
+        (xy 179.07 163.83)
+      )
+    )

Commit message: Some Tweaks
Changed lines of the file:
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@@
     (property "ki_keywords" "R res resistor")
     (attr smd)
-    (fp_text reference "R2" (at 3.175 0 90) (layer "F.SilkS")
+    (fp_text reference "R2" (at 0 -1.905 180) (layer "F.SilkS")
         (effects (font (size 1 1) (thickness 0.15)))
     )
@@
       )
     )
-  )
-  (zone (net 0) (net_name "") (layers "F&B.Cu") (name "Logo") (hatch edge 0.5)
-    (connect_pads (clearance 0))
-    (min_thickness 0.25) (filled_areas_thickness no)
-    (keepout (tracks allowed) (vias not_allowed) (pads allowed) (copperpour allowed) (footprints not_allowed))
-    (fill (thermal_gap 0.5) (thermal_bridge_width 0.5))
-    (polygon
-      (pts
-        (xy 229.87 163.83)
-        (xy 229.87 148.59)
-        (xy 210.82 148.59)
-        (xy 210.82 156.21)
-        (xy 179.07 156.21)
-        (xy 179.07 163.83)
-      )
-    )
