File: [EXOTIC] AVR Kit D7 Placed Beside Rest D.kicad_pcb (KiCad board)
At the start: 2 copper layers, 105 x 80 mm, 56 parts, among them J1 Barrel_Jack_Switch, J2 AVR-ISP-10, J3 USB_B, J4 Port A, J5 Port B, J6 Port C + D7, J7 Port D, J8 5V Headers, J9 3.3 V Headers, Q1 AO3401A, Q2 SI2302, SW1 SW_Push, SW2 SW_DPDT_x2, U1 ATmega32A-P, U2 AMS1117-5.0, U3 AMS1117-3.3, U4 LM324, U5 LM339, U6 CH340C, Y1 16 MHz

Commit message: New Subrevision
Parts:
- removed the G*** at (130.8, 77.5)
- added G***: LOGO, M's Library:TeamExotic_Logo_H40mm, B.Cu at (203.9, 109.6)
- added R12: 0 Ω, Resistor_SMD:R_1206_3216Metric_Pad1.30x1.75mm_HandSolder, F.Cu at (134.6, 105.4)
- added R13: 0 Ω, Resistor_SMD:R_1206_3216Metric_Pad1.30x1.75mm_HandSolder, F.Cu at (134.6, 100.0)
- J6: value Port C + D7 -> Port C; footprint Connector_PinSocket_2.54mm:PinSocket_1x09_P2.54mm_Vertical -> Connector_PinSocket_2.54mm:PinSocket_1x08_P2.54mm_Vertical
- J7: footprint Connector_PinSocket_2.54mm:PinSocket_1x07_P2.54mm_Vertical -> Connector_PinSocket_2.54mm:PinSocket_1x08_P2.54mm_Vertical
- moved R1 3.81 mm to (130.8, 95.2)
- moved R11 3.81 mm to (130.8, 101.6)
- moved C11 2.54 mm to (133.3, 81.3)
- moved C12 2.54 mm to (130.8, 81.3)
- moved J6 2.54 mm to (141.0, 120.7)
- moved R2 1.91 mm to (196.8, 59.7)
- moved J2 1.27 mm to (123.2, 99.1)
- moved C5 0.08 mm to (172.7, 71.2)
Connections:
- J6 pad 1: /PD7 -> /SCL
- J6 pad 2: /SCL -> /SDA
- J6 pad 3: /SDA -> /TCK
- J6 pad 4: /TCK -> /TMS
- J6 pad 5: /TMS -> /TDO
- J6 pad 6: /TDO -> /TDI
- J6 pad 7: /TDI -> /PC6
- J6 pad 8: /PC6 -> /PC7
Routing:
- net Net-(J7-Pin_8): track 0.00 -> 11.4 mm
- net /MOSI: track 72.6 -> 80.0 mm
- net -V_{In}: track 123.6 -> 117.9 mm
- net +5V: track 207.5 -> 211.4 mm
- net Net-(R12-Pad2): track 0.00 -> 2.26 mm
- net /~{RESET}: track 232.7 -> 230.7 mm
- net +5V_{NetTie}: track 68.1 -> 66.1 mm
- net Net-(U4D--): track 10.3 -> 8.43 mm
- net /SCK: track 173.6 -> 171.8 mm
- net /MISO: track 158.8 -> 157.5 mm
- net /PD7: track 11.0 -> 12.2 mm
- net Net-(U4A--): track 16.2 -> 15.3 mm
- net GND: vias 17 -> 15
Other:
- board text added: "D7"
