File: [EXOTIC] AVR Kit Flipped Port C.kicad_pcb (KiCad board)
At the start: 2 copper layers, 105 x 80 mm, 56 parts, among them J1 Barrel_Jack_Switch, J2 AVR-ISP-10, J3 USB_B, J4 Port A, J5 Port B, J6 Port C + D7, J7 Port D, J8 5V Headers, J9 3.3 V Headers, Q1 AO3401A, Q2 SI2302, SW1 SW_Push, SW2 SW_DPDT_x2, U1 ATmega32A-P, U2 AMS1117-5.0, U3 AMS1117-3.3, U4 LM324, U5 LM339, U6 CH340C, Y1 16 MHz

Commit message: New Subrevision
Parts:
- removed the G*** at (130.8, 77.5)
- added G***: LOGO, M's Library:TeamExotic_Logo_H40mm, B.Cu at (203.9, 109.6)
- moved J6 20.3 mm to (158.8, 120.7), turned to -90 degrees
- moved R2 1.91 mm to (196.8, 59.7)
- moved C5 0.08 mm to (172.7, 71.2)
Routing:
- net /TMS: track 11.0 -> 44.3 mm
- net /PC7: track 11.0 -> 43.5 mm
- net /TCK: track 11.0 -> 39.2 mm
- net /PC6: track 11.0 -> 38.9 mm
- net /TDI: track 11.0 -> 34.8 mm
- net /SDA: track 11.0 -> 34.2 mm
- net /TDO: track 11.0 -> 29.8 mm
- net /SCL: track 11.0 -> 29.1 mm
- net /PD7: track 11.0 -> 19.7 mm
- net -V_{In}: track 123.6 -> 117.9 mm
- net Net-(U4D--): track 10.3 -> 8.43 mm
- net /MISO: track 158.8 -> 159.9 mm
- net +5V_{NetTie}: track 68.1 -> 69.1 mm
- net /SCK: track 173.6 -> 174.7 mm
- net Net-(U4A--): track 16.2 -> 15.3 mm
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