File: [EXOTIC] AVR Kit Flipped Port C.kicad_sch (KiCad schematic)
At the start: 24 parts, among them J2 AVR-ISP-10, J3 USB_B, J4 Port A, J5 Port B, J6 Port C + D7, J7 Port D, SW1 SW_Push, U1 ATmega32A-P, U6 CH340C, Y1 16 MHz

Commit message: New Subrevision
Connections:
- net PC6: now also J6.7 (Pin_7); no longer J6.8 (Pin_8)
- net PC7: now also J6.8 (Pin_8); no longer J6.9 (Pin_9)
- net PD7: now also J6.9 (Pin_9); no longer J6.1 (Pin_1)
- net SCL: now also J6.1 (Pin_1); no longer J6.2 (Pin_2)
- net SDA: now also J6.2 (Pin_2); no longer J6.3 (Pin_3)
- net TCK: now also J6.3 (Pin_3); no longer J6.4 (Pin_4)
- net TDI: now also J6.6 (Pin_6); no longer J6.7 (Pin_7)
- net TDO: now also J6.5 (Pin_5); no longer J6.6 (Pin_6)
- net TMS: now also J6.4 (Pin_4); no longer J6.5 (Pin_5)
Changed lines of the file:
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@@
     (effects (font (size 1.27 1.27)) (justify left bottom))
   )
-  (label "SCL" (at 196.85 113.03 0) (fields_autoplaced)
+  (label "SCL" (at 196.85 110.49 0) (fields_autoplaced)
     (effects (font (size 1.27 1.27)) (justify left bottom))
   )
@@
     (effects (font (size 1.27 1.27)) (justify left bottom))
   )
-  (label "TCK" (at 196.85 118.11 0) (fields_autoplaced)
+  (label "TCK" (at 196.85 115.57 0) (fields_autoplaced)
     (effects (font (size 1.27 1.27)) (justify left bottom))
   )
-  (label "TMS" (at 196.85 120.65 0) (fields_autoplaced)
+  (label "TMS" (at 196.85 118.11 0) (fields_autoplaced)
     (effects (font (size 1.27 1.27)) (justify left bottom))
   )
@@
     (effects (font (size 1.27 1.27)) (justify left bottom))
   )
-  (label "PD7" (at 196.85 110.49 0) (fields_autoplaced)
+  (label "PD7" (at 196.85 130.81 0) (fields_autoplaced)
     (effects (font (size 1.27 1.27)) (justify left bottom))
   )
-  (label "PC6" (at 196.85 128.27 0) (fields_autoplaced)
+  (label "PC6" (at 196.85 125.73 0) (fields_autoplaced)
     (effects (font (size 1.27 1.27)) (justify left bottom))
   )
@@
     (effects (font (size 1.27 1.27)) (justify left bottom))
   )
-  (label "TDI" (at 196.85 125.73 0) (fields_autoplaced)
+  (label "TDI" (at 196.85 123.19 0) (fields_autoplaced)
     (effects (font (size 1.27 1.27)) (justify left bottom))
   )
@@
     (effects (font (size 1.27 1.27)) (justify left bottom))
   )
-  (label "SDA" (at 196.85 115.57 0) (fields_autoplaced)
+  (label "SDA" (at 196.85 113.03 0) (fields_autoplaced)
     (effects (font (size 1.27 1.27)) (justify left bottom))
   )
@@
     (effects (font (size 1.27 1.27)) (justify left bottom))
   )
-  (label "PC7" (at 196.85 130.81 0) (fields_autoplaced)
+  (label "PC7" (at 196.85 128.27 0) (fields_autoplaced)
     (effects (font (size 1.27 1.27)) (justify left bottom))
   )
@@
     (effects (font (size 1.27 1.27)) (justify left bottom))
   )
-  (label "TDO" (at 196.85 123.19 0) (fields_autoplaced)
+  (label "TDO" (at 196.85 120.65 0) (fields_autoplaced)
     (effects (font (size 1.27 1.27)) (justify left bottom))
   )
