File: Power Management Circuitry Original.kicad_sch (KiCad schematic)
At the start: 19 parts, among them J1 Barrel_Jack_Switch, J8 5V Headers, J9 3.3 V Headers, Q1 AO3401A, SW2 SW_DPDT_x2, U2 AMS1117-3.3, U3 AMS1117-5.0, U4 LM324

Commit message: Pre Rev. 4
Parts:
- removed R11 (x2): 0 Ω, Resistor_SMD:R_1206_3216Metric_Pad1.30x1.75mm_HandSolder, symbol Device:R
- removed unit 3 of U4
- added Q2: SI2302, Package_TO_SOT_SMD:SOT-23_Handsoldering, symbol M's Library:SI2302
- added R10 (x2): 0 Ω, Resistor_SMD:R_1206_3216Metric_Pad1.30x1.75mm_HandSolder, symbol Device:R
- added R3 (x2): 10 kΩ, Resistor_SMD:R_1206_3216Metric_Pad1.30x1.75mm_HandSolder, symbol Device:R
- added R4: 330 kΩ, Resistor_SMD:R_1206_3216Metric_Pad1.30x1.75mm_HandSolder, symbol Device:R
- added R7: 0.1 Ω, Resistor_SMD:R_1206_3216Metric_Pad1.30x1.75mm_HandSolder, symbol Device:R
- added RV1, RV2, RV3: 10 kΩ, Potentiometer_THT:Potentiometer_Bourns_3296W_Vertical, symbol Device:R_Potentiometer
- added unit 1 of U4
- added unit 2 of U4
- added unit 4 of U4
- added U5: LM339, Package_SO:SOIC-14_3.9x8.7mm_P1.27mm, symbol Comparator:LM339
- renumbered R5 to R6
Connections:
- net +5V_{PPTC} is gone; now on net +5V: R11.1
- net +3V3: now also R10.2
- net +5V: now also R3.2, R7.1, RV1.1, U5.3 (V+); no longer C8.1, J8.1 (Pin_1), J8.2 (Pin_2), U3.2 (VO), U4.4 (V+)
- net +V_{In}: now also U4.4 (V+); no longer R4.2
- net -V_{In}: now also U4.11 (V-), Q2.2 (S), R3.1, RV2.1, RV3.1
- net GND: now also Q2.3 (D), U5.12 (V-); no longer U4.11 (V-)
- net at Q1.1 (G): now also R3.1, U5.14
- net at F1.1: now also SW2.5 (B); no longer SW2.2 (B)
- net V_{In} (Unfused): now reaches J1.1
- net V_{In} (Unfused): now also R4.2, SW2.6 (C), U5.9 (+); no longer SW2.3 (C)
- new net: RV3.2, U4.12 (+)
- new net: R4.2, U4.1, U4.13 (-)
- new net: R3.2, R4.1, U4.2 (-)
- new net: RV1.3, U4.3 (+), U4.7
- new net: R10.1, U5.8 (-)
- new net: RV2.2, U4.5 (+)
- new net: RV1.2, U4.6 (-)
- new net: Q2.1 (G), U4.14
- new net: R10.1, R10.2
- new net +5V_{OCP}: C8.1, J8.1 (Pin_1), J8.2 (Pin_2), R7.2, RV2.3, RV3.3, U3.2 (VO)
