File: Unplaced Units.kicad_sch (KiCad schematic)
At the start: 4 parts, among them SW2 SW_DPDT_x2, U4 LM324

Commit message: Rev 3.99
Parts:
- removed U4 (x3): LM324, Package_SO:SO-14_3.9x8.65mm_P1.27mm, symbol Amplifier_Operational:LM324
Connections:
- no-connect marks 12 -> 3
Changed lines of the file:
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@@
     (comment 1 "Author: Morad Tamer")
   )
-  (no_connect (at 30.48 59.69))
   (no_connect (at 77.47 57.15))
   (no_connect (at 67.31 54.61))
-  (no_connect (at 45.72 74.93))
-  (no_connect (at 30.48 35.56))
   (no_connect (at 67.31 59.69))
-  (no_connect (at 45.72 38.1))
-  (no_connect (at 30.48 40.64))
-  (no_connect (at 30.48 72.39))
-  (no_connect (at 30.48 54.61))
-  (no_connect (at 30.48 77.47))
-  (no_connect (at 45.72 57.15))
   (symbol (lib_id "Switch:SW_DPDT_x2") (at 72.39 57.15 0) (mirror y) (unit 1)
     (in_bom yes) (on_board yes) (dnp no) (fields_autoplaced)
@@
         )
       )
-    )
-  )
-  (symbol (lib_id "Amplifier_Operational:LM324") (at 38.1 38.1 0) (unit 3)
-    (in_bom yes) (on_board yes) (dnp no) (fields_autoplaced)
-    (property "Reference" "U4" (at 38.1 27.94 0)
-      (effects (font (size 1.27 1.27)))
-    )
-    (property "Value" "LM324" (at 38.1 30.48 0)
-      (effects (font (size 1.27 1.27)))
-    )
-    (property "Footprint" "Package_SO:SO-14_3.9x8.65mm_P1.27mm" (at 36.83 35.56 0)
-      (effects (font (size 1.27 1.27)) hide)
-    )
-    (property "Datasheet" "http://www.ti.com/lit/ds/symlink/lm2902-n.pdf" (at 39.37 33.02 0)
-      (effects (font (size 1.27 1.27)) hide)
-    )
-    (property "Local Seller" "https://makerselectronics.com/product/lm324-sop-14-operational-amplifier-smd" (at 38.1 38.1 0)
-      (effects (font (size 1.27 1.27)) hide)
-    )
-    (pin "1")
-    (pin "2")
-    (pin "3")
-    (pin "5")
-    (pin "6")
-    (pin "7")
-    (pin "10")
-    (pin "8")
-    (pin "9")
-    (pin "12")
-    (pin "13")
-    (pin "14")
-    (pin "11")
-    (pin "4")
-    (instances
-      (project "[EXOTIC] AVR Kit"
-        (path "/bd689b4b-40d7-46ba-91b6-965ce30f8212/9da448d2-dd3c-46c7-b716-b331cd5a4621"
-          (reference "U4") (unit 3)
-        )
-        (path "/bd689b4b-40d7-46ba-91b6-965ce30f8212/9da448d2-dd3c-46c7-b716-b331cd5a4621/bbc5b563-1e1e-48b3-9d6e-3409d51ecb1f"
-          (reference "U4") (unit 1)
-        )
-      )
-    )
-  )
-  (symbol (lib_id "Amplifier_Operational:LM324") (at 38.1 57.15 0) (unit 3)
-    (in_bom yes) (on_board yes) (dnp no) (fields_autoplaced)
-    (property "Reference" "U4" (at 38.1 46.99 0)
-      (effects (font (size 1.27 1.27)))
-    )
-    (property "Value" "LM324" (at 38.1 49.53 0)
-      (effects (font (size 1.27 1.27)))
-    )
-    (property "Footprint" "Package_SO:SO-14_3.9x8.65mm_P1.27mm" (at 36.83 54.61 0)
-      (effects (font (size 1.27 1.27)) hide)
-    )
-    (property "Datasheet" "http://www.ti.com/lit/ds/symlink/lm2902-n.pdf" (at 39.37 52.07 0)
-      (effects (font (size 1.27 1.27)) hide)
-    )
-    (property "Local Seller" "https://makerselectronics.com/product/lm324-sop-14-operational-amplifier-smd" (at 38.1 57.15 0)
-      (effects (font (size 1.27 1.27)) hide)
-    )
-    (pin "1")
-    (pin "2")
-    (pin "3")
-    (pin "5")
-    (pin "6")
-    (pin "7")
-    (pin "10")
-    (pin "8")
-    (pin "9")
-    (pin "12")
-    (pin "13")
-    (pin "14")
-    (pin "11")
-    (pin "4")
-    (instances
-      (project "[EXOTIC] AVR Kit"
-        (path "/bd689b4b-40d7-46ba-91b6-965ce30f8212/9da448d2-dd3c-46c7-b716-b331cd5a4621"
-          (reference "U4") (unit 3)
-        )
-        (path "/bd689b4b-40d7-46ba-91b6-965ce30f8212/9da448d2-dd3c-46c7-b716-b331cd5a4621/bbc5b563-1e1e-48b3-9d6e-3409d51ecb1f"
-          (reference "U4") (unit 2)
-        )
-      )
-    )
-  )
-  (symbol (lib_id "Amplifier_Operational:LM324") (at 38.1 74.93 0) (unit 3)
-    (in_bom yes) (on_board yes) (dnp no) (fields_autoplaced)
-    (property "Reference" "U4" (at 38.1 64.77 0)
-      (effects (font (size 1.27 1.27)))
-    )
-    (property "Value" "LM324" (at 38.1 67.31 0)
-      (effects (font (size 1.27 1.27)))
-    )
-    (property "Footprint" "Package_SO:SO-14_3.9x8.65mm_P1.27mm" (at 36.83 72.39 0)
-      (effects (font (size 1.27 1.27)) hide)
-    )
-    (property "Datasheet" "http://www.ti.com/lit/ds/symlink/lm2902-n.pdf" (at 39.37 69.85 0)
-      (effects (font (size 1.27 1.27)) hide)
-    )
-    (property "Local Seller" "https://makerselectronics.com/product/lm324-sop-14-operational-amplifier-smd" (at 38.1 74.93 0)
-      (effects (font (size 1.27 1.27)) hide)
-    )
-    (pin "1")
-    (pin "2")
-    (pin "3")
-    (pin "5")
-    (pin "6")
-    (pin "7")
-    (pin "10")
-    (pin "8")
-    (pin "9")
-    (pin "12")
-    (pin "13")
-    (pin "14")
-    (pin "11")
-    (pin "4")
-    (instances
-      (project "[EXOTIC] AVR Kit"
-        (path "/bd689b4b-40d7-46ba-91b6-965ce30f8212/9da448d2-dd3c-46c7-b716-b331cd5a4621"
-          (reference "U4") (unit 3)
-        )
-        (path "/bd689b4b-40d7-46ba-91b6-965ce30f8212/9da448d2-dd3c-46c7-b716-b331cd5a4621/bbc5b563-1e1e-48b3-9d6e-3409d51ecb1f"
-          (reference "U4") (unit 4)
-        )
-      )
