File: Unplaced Units.kicad_sch (KiCad schematic)
At the start: 1 part, among them SW2 SW_DPDT_x2

Commit message: Rev. L4.2
Parts:
- added U4: LM339, Package_SO:SOIC-14_3.9x8.7mm_P1.27mm, symbol Comparator:LM339
Connections:
- no-connect marks 3 -> 12
Other:
- note added: "To Do: ~Priority Switch to select which 5V source is the dominant~ DONE"
- note added: "http://store.logicneed.com/product/20510"
- note added: "~Two Seperate Op-Amps needed due to difference in power source requirements (Rail selector won't work if the op amp is powered from the +12V)~ DONE"
- moved on the sheet: SW2B
