File: [EXOTIC] AVR Kit o.kicad_sch (KiCad schematic)
At the start: 21 parts, among them J2 AVR-ISP-10, J3 USB_B, J4 Port A, J5 Port B, J6 Port C + D7, J7 Port D, SW1 SW_Push, U1 ATmega32A-P, U6 CH340C, Y1 16 MHz

Commit message: Add files via upload
Parts:
- added H1, H2, H3, H4: MountingHole, MountingHole:MountingHole_2.2mm_M2_Pad, symbol Mechanical:MountingHole
Other:
- note added: "Mounting Holes"
- note removed: "Add QFN Package to the footprint"
- note removed: "Consider Ceramic Resonators"
- moved on the sheet: J4, J5, J6, J7
